File: reference_module.sch (EAGLE design)
At the start: 96 parts, among them IC1 LM324N, IC2 LM741P, IC3 LM741P, IC4 7812T, IC5 7812T

Commit message: Board file
Component placing done.
Parts:
- added C16, C17: 0.1UF/100V, amit_rcl:C-EU102-054X133
- C11, C15: value 1UF/63V -> 0.1UF/100V; device amit_rcl:CPOL-USE3.5-10 -> amit_rcl:C-EU102-054X133
Connections:
- removed net N$56: D28.A, RV8.E, S1-1.2, S1-2.2, S1-3.2
- new net N$68: C16.2, D28.A, RV8.E, S1-1.1, S1-2.1, S1-3.1
- net N$20: now also X1-14.KL
- net N$31: now also S1-8.2; no longer S1-8.1
- net N$32: now also S1-8.1; no longer S1-8.2
- net N$38: now also S1-7.2; no longer S1-7.1
- net N$40: now also S1-6.2; no longer S1-6.1
- net N$41: now also S1-6.1, S1-7.1; no longer S1-6.2, S1-7.2
- net N$47: now also C15.2, S1-2.2; no longer C15.-, S1-2.1
- net N$48: now also C11.1, C17.1; no longer C11.+
- net N$49: now also C11.2, S1-4.2; no longer C11.-, S1-4.1
- net N$54: now also C17.2, S1-4.1; no longer S1-4.2
- net N$55: now also C15.1, C16.1, S1-1.2; no longer C15.+, S1-1.1
- net N$57: now also S1-3.2, S1-5.1; no longer S1-3.1, S1-5.2
- net N$59: now also S1-5.2; no longer S1-5.1
Other:
- moved on the sheet: S1-1, S1-2, S1-3, S1-4, S1-5, S1-6, S1-7, S1-8

Commit message: schematic and PCB
changed D26 connection
added +vcc and -vcc to IC
schematic verified.
PCB layout done in diptrace.
Parts:
- removed S1: (no value), switch-dil:DIP08S
- added SW1: (no value), switch-dil:DIP08S
Connections:
- removed net N$10: C1.-, C12.2, C13.2, C2.-, C4.+, C5.2, C6.2, C8.2, D10.C, D2.A, D23.C, D24.A, D25.A, D26.A, D4.A, D9.A, IC1D.+IN, IC4.GND, IC5.VO, R20.1, RV2.E, RV4.E, RV8.A, X1-10.KL, X1-15.KL, X1-21.KL, X1-3.KL, ZD1.C
- removed net N$26: C2.+, D11.C, D13.C, D15.C, D17.C, D19.C, D21.C, D29.C, D31.C, D9.C, IC4.VO, X1-19.KL, X1-20.KL
- new net +VCC: C2.+, D11.C, D13.C, D15.C, D17.C, D19.C, D21.C, D29.C, D31.C, D9.C, IC1P.V+, IC2.V+, IC3.V+, IC4.VO, X1-19.KL, X1-20.KL
- new net -VCC: C1.-, C12.2, C13.2, C2.-, C4.+, C5.2, C6.2, C8.2, D10.C, D2.A, D23.C, D24.A, D25.A, D26.C, D4.A, D9.A, IC1D.+IN, IC1P.V-, IC2.V-, IC3.V-, IC4.GND, IC5.VO, R20.1, RV2.E, RV4.E, RV8.A, X1-10.KL, X1-15.KL, X1-21.KL, X1-3.KL, ZD1.C
- net N$31: now also SW1-8.2; no longer S1-8.2
- net N$32: now also SW1-8.1; no longer S1-8.1
- net N$38: now also SW1-7.2; no longer S1-7.2
- net N$40: now also SW1-6.2; no longer S1-6.2
- net N$41: now also SW1-6.1, SW1-7.1; no longer S1-6.1, S1-7.1
- net N$47: now also SW1-2.2; no longer S1-2.2
- net N$49: now also SW1-4.2; no longer S1-4.2
- net N$54: now also D26.A, SW1-4.1; no longer D26.C, S1-4.1
- net N$55: now also SW1-1.2; no longer S1-1.2
- net N$57: now also SW1-3.2, SW1-5.1; no longer S1-3.2, S1-5.1
- net N$59: now also SW1-5.2; no longer S1-5.2
- net N$68: now also SW1-1.1, SW1-2.1, SW1-3.1; no longer S1-1.1, S1-2.1, S1-3.1
Other:
- moved on the sheet: C11, C12, C13, C14, C15, C16, C17, D25, D26, D27, D28, D29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
